Commit message: added friction

File: src/my_bot/description/gazebo_control.xacro (robot description, xacro)
@@ -2,8 +2,8 @@
 <robot xmlns:xacro="http://www.ros.org/wiki/xacro">
     <gazebo>
-        <plugin name="diff_drive" filename="libgazebo_ros_diff_drive.so">
+        <plugin name='skid_steer_drive' filename='libgazebo_ros_skid_steer_drive.so'>
             <!-- Wheel Information -->
-            <left_joint>left_wheel_1_joint</left_joint>
-            <right_joint>right_wheel_1_joint</right_joint>
+            <left_joint>left_wheel_joint1 left_wheel_joint2 left_wheel_joint3</left_joint>
+            <right_joint>right_wheel_joint1 right_wheel_joint2 right_wheel_joint3</right_joint>
             <wheel_separation>0.35</wheel_separation>
             <wheel_diameter>0.1</wheel_diameter>

File: src/my_bot/description/robot_core.xacro (robot description, xacro)
@@ -55,4 +55,12 @@
                 <cylinder radius="0.05" length="0.04"/>
             </geometry>
+            <surface>
+                <friction>
+                    <ode>
+                        <mu>1.0</mu>
+                        <mu2>0.5</mu2>
+                    </ode>
+                </friction>
+            </surface>
         </collision>
         <xacro:inertial_cylinder mass="0.1" length="0.04" radius="0.05">
@@ -78,4 +86,12 @@
                 <cylinder radius="0.05" length="0.04"/>
             </geometry>
+            <surface>
+                <friction>
+                    <ode>
+                        <mu>1.0</mu>
+                        <mu2>0.5</mu2>
+                    </ode>
+                </friction>
+            </surface>
         </collision>
         <xacro:inertial_cylinder mass="0.1" length="0.04" radius="0.05">
@@ -101,4 +117,12 @@
                 <cylinder radius="0.05" length="0.04"/>
             </geometry>
+            <surface>
+                <friction>
+                    <ode>
+                        <mu>1.0</mu>
+                        <mu2>0.5</mu2>
+                    </ode>
+                </friction>
+            </surface>
         </collision>
         <xacro:inertial_cylinder mass="0.1" length="0.04" radius="0.05">
@@ -111,6 +135,6 @@
         <parent link="chassis"/>
         <child link="right_wheel_1"/>
-        <origin xyz="0.4 -0.175 0" rpy="-1.5708 0 0"/>
-        <axis xyz="0 0 -1"/>
+        <origin xyz="0.4 -0.175 0" rpy="1.5708 0 0"/>
+        <axis xyz="0 0 1"/>
     </joint>
     <link name="right_wheel_1">
@@ -125,4 +149,12 @@
                 <cylinder radius="0.05" length="0.04"/>
             </geometry>
+            <surface>
+                <friction>
+                    <ode>
+                        <mu>1.0</mu>
+                        <mu2>0.5</mu2>
+                    </ode>
+                </friction>
+            </surface>
         </collision>
         <xacro:inertial_cylinder mass="0.1" length="0.04" radius="0.05">
@@ -134,6 +166,6 @@
         <parent link="chassis"/>
         <child link="right_wheel_2"/>
-        <origin xyz="0.1 -0.175 0" rpy="-1.5708 0 0"/>
-        <axis xyz="0 0 -1"/>
+        <origin xyz="0.1 -0.175 0" rpy="1.5708 0 0"/>
+        <axis xyz="0 0 1"/>
     </joint>
     <link name="right_wheel_2">
@@ -148,4 +180,12 @@
                 <cylinder radius="0.05" length="0.04"/>
             </geometry>
+            <surface>
+                <friction>
+                    <ode>
+                        <mu>1.0</mu>
+                        <mu2>0.5</mu2>
+                    </ode>
+                </friction>
+            </surface>
         </collision>
         <xacro:inertial_cylinder mass="0.1" length="0.04" radius="0.05">
@@ -157,6 +197,6 @@
         <parent link="chassis"/>
         <child link="right_wheel_3"/>
-        <origin xyz="0.7 -0.175 0" rpy="-1.5708 0 0"/>
-        <axis xyz="0 0 -1"/>
+        <origin xyz="0.7 -0.175 0" rpy="1.5708 0 0"/>
+        <axis xyz="0 0 1"/>
     </joint>
     <link name="right_wheel_3">
@@ -171,4 +211,12 @@
                 <cylinder radius="0.05" length="0.04"/>
             </geometry>
+            <surface>
+                <friction>
+                    <ode>
+                        <mu>1.0</mu>
+                        <mu2>0.5</mu2>
+                    </ode>
+                </friction>
+            </surface>
         </collision>
         <xacro:inertial_cylinder mass="0.1" length="0.04" radius="0.05">
